File: kicad/_saved_wasserschaden.sch (KiCad schematic (older format))
At the start: 13 parts, among them J1 valve out, J2 12V in, U1 stepdown, U2 WeMos_mini

Commit message: added deepsleep jumper to schematic &cleanup
Parts:
- added JP1: SolderJumper_2_Open, symbol Jumper:SolderJumper_2_Open
- D1: footprint Diodes_THT:D_5KPW_P12.70mm_Horizontal -> Diodes_THT:D_A-405_P7.62mm_Horizontal; symbol D -> wasserschaden-cache-2018-10-17-20-35-24:D
- D2, D3, D4: symbol LED -> wasserschaden-cache-2018-10-17-20-35-24:LED
- IRFZ44N1: symbol 2N7000 -> wasserschaden-cache-2018-10-17-20-35-24:2N7000
- J1, J2: symbol Screw_Terminal_01x02 -> wasserschaden-cache-2018-10-17-20-35-24:Screw_Terminal_01x02
- R1, R2, R3, R4: symbol R -> wasserschaden-cache-2018-10-17-20-35-24:R
- U1: symbol stepdown -> wasserschaden-cache-2018-10-17-20-35-24:stepdown
- U2: symbol WeMos_mini -> wasserschaden-cache-2018-10-17-20-35-24:WeMos_mini
Connections:
- wire segments 13 -> 21
- no-connect marks 12 -> 10
Changed lines of the file:
@@
-EESchema Schematic File Version 2
-LIBS:power
-LIBS:device
-LIBS:switches
-LIBS:relays
-LIBS:motors
-LIBS:transistors
-LIBS:conn
-LIBS:linear
-LIBS:regul
-LIBS:74xx
-LIBS:cmos4000
-LIBS:adc-dac
-LIBS:memory
-LIBS:xilinx
-LIBS:microcontrollers
-LIBS:dsp
-LIBS:microchip
-LIBS:analog_switches
-LIBS:motorola
-LIBS:texas
-LIBS:intel
-LIBS:audio
-LIBS:interface
-LIBS:digital-audio
-LIBS:philips
-LIBS:display
-LIBS:cypress
-LIBS:siliconi
-LIBS:opto
-LIBS:atmel
-LIBS:contrib
-LIBS:valves
-LIBS:wemos_mini
-LIBS:wasserschaden-cache
-EELAYER 25 0
+EESchema Schematic File Version 4
+EELAYER 26 0
 EELAYER END
 $Descr A4 11693 8268
@@
 $EndDescr
 $Comp
-L WeMos_mini U2
+L wasserschaden-cache-2018-10-17-20-35-24:WeMos_mini U2
 U 1 1 5B26FC39
 P 4000 2100
@@
 $EndComp
 $Comp
-L 2N7000 IRFZ44N1
+L wasserschaden-cache-2018-10-17-20-35-24:2N7000 IRFZ44N1
 U 1 1 5B2A69C6
 P 2900 2250
@@
 $EndComp
 Wire Wire Line
-	3100 2250 3500 2250
-$Comp
-L Screw_Terminal_01x02 J1
+	3100 2250 3200 2250
+$Comp
+L wasserschaden-cache-2018-10-17-20-35-24:Screw_Terminal_01x02 J1
 U 1 1 5B2A6B15
 P 2450 2750
@@
 $EndComp
 $Comp
-L Screw_Terminal_01x02 J2
+L wasserschaden-cache-2018-10-17-20-35-24:Screw_Terminal_01x02 J2
 U 1 1 5B2A6B9D
 P 2450 3200
@@
 $EndComp
 $Comp
-L GND #PWR01
+L wasserschaden-cache-2018-10-17-20-35-24:GND #PWR01
 U 1 1 5B2A6BE6
 P 2650 3200
@@
 $EndComp
 $Comp
-L GND #PWR02
+L wasserschaden-cache-2018-10-17-20-35-24:GND #PWR02
 U 1 1 5B2A6C2A
 P 3500 1850
@@
 $EndComp
 $Comp
-L GND #PWR03
+L wasserschaden-cache-2018-10-17-20-35-24:GND #PWR03
 U 1 1 5B2A6C5A
 P 2800 2050
@@
 $EndComp
 $Comp
-L D D1
+L wasserschaden-cache-2018-10-17-20-35-24:D D1
 U 1 1 5B2A6D63
 P 3050 2750
 F 0 "D1" H 3050 2850 50  0000 C CNN
 F 1 " " H 3150 2850 50  0000 C CNN
-F 2 "Diodes_THT:D_5KPW_P12.70mm_Horizontal" H 3050 2750 50  0001 C CNN
+F 2 "Diodes_THT:D_A-405_P7.62mm_Horizontal" H 3050 2750 50  0001 C CNN
 F 3 "" H 3050 2750 50  0001 C CNN
 	1    3050 2750
@@
 $EndComp
 $Comp
-L stepdown U1
+L wasserschaden-cache-2018-10-17-20-35-24:stepdown U1
 U 1 1 5B2A6F8D
 P 3800 3000
@@
 	4500 1750 4950 1750
 $Comp
-L GND #PWR04
+L wasserschaden-cache-2018-10-17-20-35-24:GND #PWR04
 U 1 1 5B2A7077
 P 3400 2900
@@
 NoConn ~ 3500 2350
 NoConn ~ 3500 2450
-NoConn ~ 4500 2450
 NoConn ~ 4500 2350
-NoConn ~ 4500 2250
 NoConn ~ 4500 2150
 NoConn ~ 4500 2050
@@
 NoConn ~ 4500 1850
 Wire Wire Line
-	2650 2750 2900 2750
+	2650 2750 2800 2750
 Wire Wire Line
 	2800 2450 2800 2750
@@
 +\n-
 Wire Wire Line
-	4950 1750 4950 3050
-Wire Wire Line
 	2650 2650 3200 2650
 Wire Wire Line
 	3200 2650 3200 2750
 $Comp
-L +12V #PWR05
+L wasserschaden-cache-2018-10-17-20-35-24:+12V #PWR05
 U 1 1 5B2A7A00
 P 2650 2650
@@
 $EndComp
 $Comp
-L +12V #PWR06
+L wasserschaden-cache-2018-10-17-20-35-24:+12V #PWR06
 U 1 1 5B2A7A20
 P 2650 3100
@@
 $EndComp
 $Comp
-L +12V #PWR07
+L wasserschaden-cache-2018-10-17-20-35-24:+12V #PWR07
 U 1 1 5B2A7A40
 P 3400 3050
@@
 $EndComp
 $Comp
-L R R1
+L wasserschaden-cache-2018-10-17-20-35-24:R R1
 U 1 1 5B2A7CB0
 P 3050 2100
@@
 $EndComp
 $Comp
-L GND #PWR08
+L wasserschaden-cache-2018-10-17-20-35-24:GND #PWR08
 U 1 1 5B2A7CE4
 P 3050 1950
@@
 $EndComp
 $Comp
-L GND #PWR09
+L wasserschaden-cache-2018-10-17-20-35-24:GND #PWR09
 U 1 1 5B2A9F12
 P 4700 2900
@@
 	4950 3050 4700 3050
 $Comp
-L LED D2
+L wasserschaden-cache-2018-10-17-20-35-24:LED D2
 U 1 1 5B2BDC1C
 P 3200 1500
@@
 $EndComp
 $Comp
-L R R2
+L wasserschaden-cache-2018-10-17-20-35-24:R R2
 U 1 1 5B2BDCBD
 P 3200 1200
@@
 $EndComp
 $Comp
-L GND #PWR010
+L wasserschaden-cache-2018-10-17-20-35-24:GND #PWR010
 U 1 1 5B2BDCFD
 P 3200 1050
@@
 	-1   0    0    1
 $EndComp
-Connection ~ 4950 2000
 Wire Wire Line
 	3200 1650 3200 2250
 Connection ~ 3200 2250
 $Comp
-L LED D3
+L wasserschaden-cache-2018-10-17-20-35-24:LED D3
 U 1 1 5B2C19FD
 P 5100 2000
@@
 $EndComp
 $Comp
-L R R3
+L wasserschaden-cache-2018-10-17-20-35-24:R R3
 U 1 1 5B2C1A03
 P 5250 2150
@@
 $EndComp
 $Comp
-L GND #PWR011
+L wasserschaden-cache-2018-10-17-20-35-24:GND #PWR011
 U 1 1 5B2C1A09
 P 5250 2300
@@
 $EndComp
 $Comp
-L LED D4
+L wasserschaden-cache-2018-10-17-20-35-24:LED D4
 U 1 1 5B2C1D4C
 P 3450 1500
@@
 $EndComp
 $Comp
-L R R4
+L wasserschaden-cache-2018-10-17-20-35-24:R R4
 U 1 1 5B2C1D52
 P 3450 1200
@@
 $EndComp
 $Comp
-L GND #PWR012
+L wasserschaden-cache-2018-10-17-20-35-24:GND #PWR012
 U 1 1 5B2C1D58
 P 3450 1050
@@
 	3300 2150 3500 2150
 $Comp
-L +3.3V #PWR013
+L wasserschaden-cache-2018-10-17-20-35-24:+3V3 #PWR013
 U 1 1 5B2C1F93
 P 4950 1750
@@
 Wire Wire Line
 	3200 2250 3050 2250
+Wire Wire Line
+	2800 2750 2900 2750
+Wire Wire Line
+	3200 2250 3500 2250
+Wire Wire Line
+	4950 1750 4950 3050
+$Comp
+L Jumper:SolderJumper_2_Open JP1
+U 1 1 5BCFAE3F
+P 4750 2350
+F 0 "JP1" V 4704 2418 50  0000 L CNN
+F 1 "SolderJumper_2_Open" V 4795 2418 50  0000 L CNN
+F 2 "" H 4750 2350 50  0001 C CNN
+F 3 "~" H 4750 2350 50  0001 C CNN
+	1    4750 2350
+	0    1    1    0
+$EndComp
+Wire Wire Line
+	4750 2200 4600 2200
+Wire Wire Line
+	4600 2200 4600 2250
+Wire Wire Line
+	4600 2250 4500 2250
+Wire Wire Line
+	4500 2450 4600 2450
+Wire Wire Line
+	4600 2450 4600 2500
+Wire Wire Line
+	4600 2500 4750 2500
 $EndSCHEMATC

Commit message: cleaned up kicad dir
Parts:
- added J3: sense, Connectors_Terminal_Blocks:TerminalBlock_Altech_AK300-2_P5.00mm, symbol wasserschaden-cache-2018-10-17-20-35-24:Screw_Terminal_01x02
- added JP2: sense jumper, symbol Device:Jumper_NC_Dual
- IRFZ44N1: footprint test_wemos:irlz44n -> custom:irlz44n
- JP1: value SolderJumper_2_Open -> deepsleep jumper; footprint (none) -> custom:jumper
- U1: footprint stepdown:stepdown -> custom:stepdown
- U2: footprint test_wemos:wemos-d1-mini-with-pin-header -> custom:wemos
Connections:
- wire segments 21 -> 30
- no-connect marks 10 -> 11
Other:
- moved on the sheet: D1, D2, D4, IRFZ44N1, J1, R1, R2, R4
