File: kicad/wasserschaden_smd.sch (KiCad schematic (older format))
At the start: 18 parts, among them J1 valve out, J2 12V in, J3 sense, U1 stepdown, U2 WeMos_mini, U3 DS18B20

Commit message: pcb v7
Parts:
- D1: footprint Diodes_THT:D_A-405_P7.62mm_Horizontal -> Diodes_SMD:D_SMA_Handsoldering
- IRFZ44N1: footprint custom:irlz44n -> custom:irlz44n_vertical
Changed lines of the file:
@@
 EESchema Schematic File Version 4
+LIBS:wasserschaden_smd-cache
 EELAYER 26 0
 EELAYER END
@@
 F 0 "IRFZ44N1" H 2950 2250 50  0000 L CNN
 F 1 " " H 2900 2250 50  0000 L CNN
-F 2 "custom:irlz44n" H 2900 2175 50  0001 L CIN
+F 2 "custom:irlz44n_vertical" H 2900 2175 50  0001 L CIN
 F 3 "" H 2700 2250 50  0001 L CNN
 	1    2700 2250
@@
 F 0 "D1" H 2850 2850 50  0000 C CNN
 F 1 " " H 2950 2850 50  0000 C CNN
-F 2 "Diodes_THT:D_A-405_P7.62mm_Horizontal" H 2850 2750 50  0001 C CNN
+F 2 "Diodes_SMD:D_SMA_Handsoldering" H 2850 2750 50  0001 C CNN
 F 3 "" H 2850 2750 50  0001 C CNN
 	1    2850 2750
