File: kicad_3valves/wasserschaden.sch (KiCad schematic (older format))
At the start: 30 parts

Commit message: fancy routing for 3 valve board
Parts:
- J1, J2, J3, J4, J5: renamed from J?; footprint Connectors_Terminal_Blocks:TerminalBlock_Altech_AK300-2_P5.00mm -> custom:termina_2pin
- gave numbers to parts that had none: 25
