File: bridge_platine/bridge_platine_v1/bridge_platine_v1.kicad_pcb (KiCad board)
At the start: 2 copper layers, 27.7 x 47.8 mm, 15 parts, among them J1 Screw_Terminal_01x02, U1 stepdown-wasserschaden-cache-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, U2 WeMos_D1_mini

Commit message: added missing track
Routing:
- net Net-(1k3-Pad1): track 0.00 -> 3.59 mm
Changed lines of the file:
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@@
     (thickness 1.6)
     (drawings 5)
-    (tracks 27)
+    (tracks 28)
     (zones 0)
     (modules 15)
@@
   (segment (start 26.67 59.69) (end 26.67 64.77) (width 0.25) (layer F.Cu) (net 3))
   (segment (start 30.48 63.5) (end 34.29 59.69) (width 0.25) (layer F.Cu) (net 4))
+  (segment (start 24.13 64.77) (end 26.67 67.31) (width 0.25) (layer B.Cu) (net 5))
   (segment (start 30.48 71.12) (end 34.29 67.31) (width 0.25) (layer F.Cu) (net 6))
   (segment (start 45.293949 53.34) (end 44.304 53.34) (width 0.25) (layer F.Cu) (net 7))
